File: BlinkeShit_Example/BlinkeShit_Example.kicad_pcb (KiCad board)
At the start: 2 copper layers, 30 parts, among them J18 Con_3-5V, SW1 SW_Push

Commit message: maybe new bitbadge
Parts:
- removed the REF** at (175.0, 99.7)
- removed the REF** at (151.0, 93.7)
- removed the REF** at (175.0, 87.7)
- removed the REF** at (169.0, 87.7)
- removed the REF** at (163.0, 87.7)
- removed the REF** at (157.0, 87.7)
- removed the REF** at (151.0, 87.7)
- removed the REF** at (175.0, 81.7)
- removed the REF** at (169.0, 81.7)
- removed the REF** at (163.0, 81.7)
- removed the REF** at (157.0, 81.7)
- removed the REF** at (169.0, 99.7)
- removed the REF** at (151.0, 81.7)
- removed the REF** at (163.0, 99.7)
- removed the REF** at (157.0, 99.7)
- removed the REF** at (151.0, 99.7)
- removed the REF** at (175.0, 93.7)
- removed the REF** at (169.0, 93.7)
- removed the REF** at (163.0, 93.7)
- removed the REF** at (157.0, 93.7)
- added REF**: FlashCrap_0805, SGMK_BlinkeShit3000:FlashCrap_0805, F.Cu at (201.6, 75.0)
- added REF**: FlashCrap_0805, SGMK_BlinkeShit3000:FlashCrap_0805, F.Cu at (191.6, 70.0)
- added REF**: FlashCrap_0805, SGMK_BlinkeShit3000:FlashCrap_0805, F.Cu at (186.6, 70.0)
- added REF**: FlashCrap_0805, SGMK_BlinkeShit3000:FlashCrap_0805, F.Cu at (181.6, 70.0)
- added REF**: FlashCrap_0805, SGMK_BlinkeShit3000:FlashCrap_0805, F.Cu at (176.6, 70.0)
- added REF**: FlashCrap_0805, SGMK_BlinkeShit3000:FlashCrap_0805, F.Cu at (171.6, 70.0)
- added REF**: FlashCrap_0805, SGMK_BlinkeShit3000:FlashCrap_0805, F.Cu at (201.6, 65.0)
- added REF**: FlashCrap_0805, SGMK_BlinkeShit3000:FlashCrap_0805, F.Cu at (196.6, 65.0)
- added REF**: FlashCrap_0805, SGMK_BlinkeShit3000:FlashCrap_0805, F.Cu at (191.6, 65.0)
- added REF**: FlashCrap_0805, SGMK_BlinkeShit3000:FlashCrap_0805, F.Cu at (186.6, 65.0)
- added REF**: FlashCrap_0805, SGMK_BlinkeShit3000:FlashCrap_0805, F.Cu at (181.6, 65.0)
- added REF**: FlashCrap_0805, SGMK_BlinkeShit3000:FlashCrap_0805, F.Cu at (196.6, 75.0)
- added REF**: FlashCrap_0805, SGMK_BlinkeShit3000:FlashCrap_0805, F.Cu at (176.6, 65.0)
- added REF**: FlashCrap_0805, SGMK_BlinkeShit3000:FlashCrap_0805, F.Cu at (171.6, 65.0)
- added REF**: FlashCrap_0805, SGMK_BlinkeShit3000:FlashCrap_0805, F.Cu at (201.6, 60.0)
- added REF**: FlashCrap_0805, SGMK_BlinkeShit3000:FlashCrap_0805, F.Cu at (196.6, 60.0)
- added REF**: FlashCrap_0805, SGMK_BlinkeShit3000:FlashCrap_0805, F.Cu at (191.6, 60.0)
- added REF**: FlashCrap_0805, SGMK_BlinkeShit3000:FlashCrap_0805, F.Cu at (186.6, 60.0)
- added REF**: FlashCrap_0805, SGMK_BlinkeShit3000:FlashCrap_0805, F.Cu at (181.6, 60.0)
- added REF**: FlashCrap_0805, SGMK_BlinkeShit3000:FlashCrap_0805, F.Cu at (176.6, 60.0)
- added REF**: FlashCrap_0805, SGMK_BlinkeShit3000:FlashCrap_0805, F.Cu at (171.6, 60.0)
- added REF**: FlashCrap_0805, SGMK_BlinkeShit3000:FlashCrap_0805, F.Cu at (201.6, 55.0)
- added REF**: FlashCrap_0805, SGMK_BlinkeShit3000:FlashCrap_0805, F.Cu at (191.6, 75.0)
- added REF**: FlashCrap_0805, SGMK_BlinkeShit3000:FlashCrap_0805, F.Cu at (196.6, 55.0)
- added REF**: FlashCrap_0805, SGMK_BlinkeShit3000:FlashCrap_0805, F.Cu at (191.6, 55.0)
- added REF**: FlashCrap_0805, SGMK_BlinkeShit3000:FlashCrap_0805, F.Cu at (186.6, 55.0)
- added REF**: FlashCrap_0805, SGMK_BlinkeShit3000:FlashCrap_0805, F.Cu at (181.6, 55.0)
- added REF**: FlashCrap_0805, SGMK_BlinkeShit3000:FlashCrap_0805, F.Cu at (176.6, 55.0)
- added REF**: FlashCrap_0805, SGMK_BlinkeShit3000:FlashCrap_0805, F.Cu at (186.6, 75.0)
- added REF**: FlashCrap_0805, SGMK_BlinkeShit3000:FlashCrap_0805, F.Cu at (181.6, 75.0)
- added REF**: FlashCrap_0805, SGMK_BlinkeShit3000:FlashCrap_0805, F.Cu at (176.6, 75.0)
- added REF**: FlashCrap_0805, SGMK_BlinkeShit3000:FlashCrap_0805, F.Cu at (171.6, 75.0)
- added REF**: FlashCrap_0805, SGMK_BlinkeShit3000:FlashCrap_0805, F.Cu at (201.6, 70.0)
- added REF**: FlashCrap_0805, SGMK_BlinkeShit3000:FlashCrap_0805, F.Cu at (196.6, 70.0)
- moved REF** 62.7 mm to (171.6, 55.0), turned to 90 degrees
- moved POT1-MAIN1 45.8 mm to (99.7, 70.4)
- moved J18 37.0 mm to (162.9, 75.2)
- moved SW1 33.8 mm to (162.9, 61.6), turned to 180 degrees
- moved REF** 19.3 mm to (119.1, 90.3)
Routing:
- net (no net): track 304.5 -> 384.2 mm
